File: vusbtinyisp_smt_inline.brd (EAGLE design)
At the start: 19.7 x 29.2 mm, 9 parts, among them U1 Tiny85-20-SMT

Commit message: changing 1k to 1.5k resistors in 5V designs
Parts:
- R3: value 1k Ohm -> 1.5k Ohm
Changed lines of the file:
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@@
 <element name="R1" library="resistor" package="R0805" value="68ohm" x="52.07" y="35.56" rot="R270"/>
 <element name="R2" library="resistor" package="R0805" value="68 ohm" x="54.61" y="35.56" rot="R270"/>
-<element name="R3" library="resistor" package="R1206" value="1k Ohm" x="49.53" y="38.1" rot="R90"/>
+<element name="R3" library="resistor" package="R1206" value="1.5k Ohm" x="49.53" y="38.1" rot="R90"/>
 <element name="JP2" library="SparkFun-Connectors" package="USB-MINIB" value="USBSMD" x="53.34" y="27.94" rot="R90">
 <attribute name="PROD_ID" value="CONN-08193" x="40.64" y="16.51" size="1.016" layer="27" rot="R90" display="off"/>
