File: vusbtinyisp_smt_inline.sch (EAGLE design)
At the start: 9 parts, among them U1 Tiny85-20-SMT

Commit message: changing 1k to 1.5k resistors in 5V designs
Parts:
- R3: value 1k Ohm -> 1.5k Ohm
Changed lines of the file:
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@@
 <part name="SUPPLY3" library="supply2" deviceset="GND" device=""/>
 <part name="P+2" library="supply1" deviceset="VCC" device=""/>
-<part name="R3" library="resistor" deviceset="R-EU_" device="R1206" value="1k Ohm"/>
+<part name="R3" library="resistor" deviceset="R-EU_" device="R1206" value="1.5k Ohm"/>
 <part name="JP2" library="SparkFun-Connectors" deviceset="USB" device="SMD"/>
 <part name="U$1" library="elliot" deviceset="SMT_ISP" device=""/>
