File: vusbtinyisp_smt_voltage_reg.brd (EAGLE design)
At the start: 39.3 x 20.3 mm, 9 parts, among them IC1 MCP170333MB, U2 TINY45-20-DIP

Commit message: changing 1k to 1.5k resistors in 5V designs
Parts:
- C1, C2: value (none) -> 1uF
Changed lines of the file:
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@@
 </autorouter>
 <elements>
-<element name="C1" library="SparkFun-Passives" package="1206" value="" x="52.07" y="33.02" rot="R180"/>
+<element name="C1" library="SparkFun-Passives" package="1206" value="1uF" x="52.07" y="33.02" rot="R180"/>
 <element name="USB" library="pinhead" package="1X04" value="" x="39.878" y="38.1" rot="R270"/>
 <element name="R1" library="resistor" package="R0805" value="68ohm" x="44.45" y="39.37" rot="R180"/>
@@
 <element name="R3" library="resistor" package="R1206" value="1k Ohm" x="44.958" y="41.91"/>
 <element name="U$1" library="elliot" package="SMT_PADS" value="SMT_ISP" x="60.96" y="41.91"/>
-<element name="C2" library="SparkFun-Passives" package="1206" value="" x="36.068" y="39.37" rot="R270"/>
+<element name="C2" library="SparkFun-Passives" package="1206" value="1uF" x="36.068" y="39.37" rot="R270"/>
 <element name="IC1" library="linear" package="SOT89" value="MCP170333MB" x="31.75" y="39.37" rot="R90"/>
 <element name="U2" library="SparkFun-DigitalIC" package="DIP08" value="TINY45-20-DIP" x="53.34" y="39.37" rot="R270">
